File: kicad/cluster.sch (KiCad schematic (older format))
At the start: 16 parts, among them J1 Conn_01x07

Commit message: Added ground planes, combined left and right thumb cluster PCBs
Parts:
- R1, R2, R3, R4, R5: footprint Resistor_SMD:R_1206_3216Metric_Pad1.42x1.75mm_HandSolder -> Resistor_SMD:R_0603_1608Metric
Connections:
- wire segments 10 -> 25
Other:
- moved on the sheet: IR1, J1
